File: Kicad/equipo_medicion_ensayo_celdas.kicad_sch (KiCad schematic)
At the start: 33 parts, among them J2 Conn_Coaxial, J3 Conn_01x06, J4 USB_C_Receptacle_USB2.0_16P, SW1 SW_Push, SW2 SW_Push, U1 STM32WB55RGVx, U2 USBLC6-2SC6, X1 32.768kHz, X2 32MHz

Commit message: Más avances en esquemático de Kicad.
Parts:
- added C36, C37: 10u, symbol Device:C
- added D4, D5: B560C, symbol Device:D_Schottky
- added J1: Micro_SD_Card, symbol Connector:Micro_SD_Card
- added U6: LM1117DT-3.3, Package_TO_SOT_SMD:TO-252-3_TabPin2, symbol Regulator_Linear:LM1117DT-3.3
Connections:
- net GND: now also C36.2, C37.2, U6.1 (GND)
- net VBUS: now reaches J4.A4 (VBUS), J4.A9 (VBUS), J4.B4 (VBUS), J4.B9 (VBUS), U2.5 (VBUS)
- net VBUS: now also D5.2 (A)
- new net: C36.1, D4.1 (K), D5.1 (K), U6.3 (VI)
- new net POWER_IN/VOUT_5V: D4.2 (A)
- new net VOUT_3V3: C37.1, U6.2 (VO)
Other:
- sheet POWER_IN ports: added VIN, VOUT_5V, VOUT_9V; removed none
