File: Kicad/cell_tester_module.kicad_sch (KiCad schematic)
At the start: 13 parts, among them Q10 NPN, Q6 NPN, Q7 NPN, Q8 PNP, Q9 PNP, U2 LM358

Commit message: Más avances en el esquemático.
Parts:
- added C1: 1n, symbol Device:C
- added D5, D9: 1N4148, Diode_THT:D_DO-35_SOD27_P7.62mm_Horizontal, symbol Diode:1N4148
- added J1: Screw_Terminal_01x02, symbol Connector:Screw_Terminal_01x02
- added R31: R, symbol Device:R
- added R32: 100k, symbol Device:R
- Q10: value NPN -> TIP35C
- Q7: value NPN -> 2N2222
- Q8: value PNP -> 2N2907
- Q9: value PNP -> TIP36C
- R29: value 4K7 -> 1k
- R30: value 1K -> R
Connections:
- net +12V: no longer R18.1
- net GND: now also R32.1; no longer R30.2
- net VGND: now also R30.2; no longer Q10.1 (C), Q7.3 (E), Q8.3 (E), Q9.1 (C), U2.2 (-)
- net at Q6.3 (E), Q8.2 (B), RV2.3: now also D5.2 (A); no longer R30.1
- net at Q6.1 (C), Q7.2 (B), R29.2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: no longer U2.1
- new net: J1.1 (Pin_1), Q10.1 (C), Q7.3 (E), Q8.3 (E), Q9.1 (C)
- new net: J1.2 (Pin_2), R30.1
- new net: C1.2, D5.1 (K), U2.1
- new net: C1.1, U2.2 (-)
- new net VIN_SPLIT: R18.1
Other:
- moved on the sheet: Q10, Q7, Q8, Q9, R29
