File: Kicad/cell_tester_module.kicad_sch (KiCad schematic)
At the start: 13 parts, among them Q10 NPN, Q6 NPN, Q7 NPN, Q8 PNP, Q9 PNP, U2 LM358

Commit message: Pruebas y arreglos relacionados a compensación de lazo de tensión y mediciones de frontend de módulo de carga.
Parts:
- removed D4: 1N5221, symbol Device:D_Zener
- removed R19: 14k, symbol Device:R
- removed R20: 10k, symbol Device:R
- added C1, C2, C37: 1n, symbol Device:C
- added C13: 10n, symbol Device:C
- added C3: 1u, symbol Device:C
- added D10, D5, D9: 1N4148, Diode_THT:D_DO-35_SOD27_P7.62mm_Horizontal, symbol Diode:1N4148
- added J1, J2: Screw_Terminal_01x02, symbol Connector:Screw_Terminal_01x02
- added K7: Relay_SPDT, Relay_THT:Relay_SPDT_SANYOU_SRD_Series_Form_C, symbol Relay:Relay_SPDT
- added Q11: 2N2222, symbol Simulation_SPICE:NPN
- added R130: 270, symbol Device:R
- added R140, R34, R46: 10k, symbol Device:R
- added R31, R32, R36, R41, R42, R43, R44, R47, R48, R49, R50, R51, R54, R55: 100k, symbol Device:R
- added R33, R45: 91k, symbol Device:R
- added R35: 200k, symbol Device:R
- added R37, R38, R39: 150k, symbol Device:R
- added R40: 9k1, symbol Device:R
- added R52: 1k, symbol Device:R
- added RV3, RV5: 10k, symbol Device:R_Potentiometer_Trim
- added U10, U11, U12, U6, U9: LM358, symbol Amplifier_Operational:LM358
- added U35: MCP4822, symbol Analog_DAC:MCP4822
- Q10: value NPN -> TIP35C
- Q7: value NPN -> 2N2222
- Q8: value PNP -> 2N2907
- Q9: value PNP -> TIP36C
- R18: value 10k -> 1k
- R29: value 4K7 -> 1k
- R30: value 1K -> 100m
Connections:
- net +12V: now also U6.8 (V+); no longer Q9.3 (E), R18.1, R29.1
- net GND: now also C37.2, J2.2 (Pin_2), Q11.3 (E), U35.5 (~{LDAC}), U35.7 (Vss), U6.4 (V-); no longer Q10.3 (E), R30.2, U2.4 (V-)
- net VGND: now also R30.2, R34.2, R49.2; no longer Q10.1 (C), Q7.3 (E), Q8.3 (E), Q9.1 (C), U2.2 (-)
- net at Q6.3 (E), Q8.2 (B), RV2.3: now also D5.2 (A), D9.2 (A); no longer R30.1
- net at R18.2: now also C13.1, R37.1
- net at Q6.1 (C), Q7.2 (B), R29.2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: no longer U2.1
- net VGND_REF: no longer names the net of U2.3 (+)
- net VGND_REF: now also R35.2, U9.1
- new net: R43.2, R44.1, U10.2 (-)
- new net: R41.2, R42.1, U10.3 (+)
- new net: R55.2, RV5.1, RV5.2, U12.3 (+)
- new net: C2.2, D9.1 (K), U6.1
- new net: C2.1, R40.1, U6.2 (-)
- new net: R33.2, R34.1, U6.3 (+)
- new net: R48.1, R51.2, RV3.1, RV3.2
- new net: R49.1, R50.2, U11.2 (-)
- new net: R47.1, R48.2, U11.3 (+)
- new net: Q11.2 (B), R130.1
- new net: R37.2, R38.2, R39.1, U9.3 (+)
- new net: J1.1 (Pin_1), K7.14, R31.2, R42.2
- new net: J1.2 (Pin_2), R30.1, R38.1, R40.2, R44.2, R47.2
- new net: C37.1, D10.2 (A), K7.A1, Q11.1 (C)
- new net: R35.1, R36.2, U9.2 (-)
- new net: K7.11, Q10.1 (C), Q7.3 (E), Q8.3 (E), Q9.1 (C)
- new net: R33.1, U35.6 (VB)
- new net: C3.1, R45.2, R46.1
- new net: R52.1, R54.2, U12.2 (-)
- new net: C3.2, R52.2
- new net: R18.1, U35.8 (VA)
- new net: C1.1, R31.1, R32.2, U2.2 (-)
- new net: C1.2, D5.1 (K), U2.1
- new net +5V: D10.1 (K), K7.A2, R140.1, U35.1 (Vdd)
- new net BAT_POW_EN: R130.2
- new net IBAT_ADC: R50.1, U11.1
- new net MCP_NCS: U35.2 (~{CS})
- new net MCP_SCK: U35.3 (SCK)
- new net MCP_SDI: U35.4 (SDI)
- new net TBAT_ADC: J2.1 (Pin_1), R140.2
- new net VBAT_AC_ADC: R54.1, U12.1
- new net VBAT_ADC: R43.1, R45.1, U10.1
- new net VCC+: Q9.3 (E), R29.1, R51.1, R55.1, U10.8 (V+), U11.8 (V+), U12.8 (V+), U9.8 (V+)
- new net VCC-: C13.2, Q10.3 (E), R32.1, R36.1, R39.2, R41.1, R46.2, RV3.3, RV5.3, U10.4 (V-), U11.4 (V-), U12.4 (V-), U2.4 (V-), U9.4 (V-)
- no-connect marks 0 -> 1
Other:
- note added: "BAT Connection Terminal"
- note added: "R = (3V3 - 0.7V)/I_Coil*hfe_sat = (3V3 - 0.7V)/100mA*10 = 260"
- note added: "Temperature NTC"
- moved on the sheet: Q10, Q6, Q7, Q8, Q9, R29, RV2, U2A, U2C

Commit message: Correcciones y mejoras en esquemático y simulaciones.
Parts:
- C1: value 1n -> 330n
Connections:
- net VCC-: no longer R32.1
- net at J1.2 (Pin_2), R30.1, R38.1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: now also R32.1
Changed lines of the file:
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@@
 	)
 	(junction
-		(at 220.98 148.59)
-		(diameter 0)
-		(color 0 0 0 0)
-	)
-	(junction
 		(at 77.47 50.8)
 		(diameter 0)
@@
 	)
 	(junction
+		(at 138.43 163.83)
+		(diameter 0)
+		(color 0 0 0 0)
+	)
+	(junction
 		(at 266.7 87.63)
 		(diameter 0)
@@
 	(wire
 		(pts
-			(xy 138.43 148.59) (xy 220.98 148.59)
-		)
-		(stroke
-			(width 0)
-			(type default)
-		)
-	)
-	(wire
-		(pts
 			(xy 77.47 50.8) (xy 77.47 55.88)
 		)
@@
 	(wire
 		(pts
+			(xy 259.08 135.89) (xy 259.08 163.83)
+		)
+		(stroke
+			(width 0)
+			(type default)
+		)
+	)
+	(wire
+		(pts
 			(xy 342.9 142.24) (xy 342.9 147.32)
 		)
@@
 	(wire
 		(pts
-			(xy 138.43 128.27) (xy 138.43 148.59)
+			(xy 138.43 128.27) (xy 138.43 163.83)
 		)
 		(stroke
@@
 	(wire
 		(pts
-			(xy 220.98 138.43) (xy 220.98 148.59)
+			(xy 220.98 138.43) (xy 220.98 153.67)
 		)
 		(stroke
@@
 	(wire
 		(pts
-			(xy 99.06 163.83) (xy 259.08 163.83)
+			(xy 99.06 163.83) (xy 138.43 163.83)
 		)
 		(stroke
@@
 	(wire
 		(pts
-			(xy 220.98 148.59) (xy 220.98 153.67)
-		)
-		(stroke
-			(width 0)
-			(type default)
-		)
-	)
-	(wire
-		(pts
 			(xy 322.58 114.3) (xy 322.58 116.84)
 		)
@@
 	(wire
 		(pts
-			(xy 259.08 135.89) (xy 259.08 163.83)
-		)
-		(stroke
-			(width 0)
-			(type default)
-		)
-	)
-	(wire
-		(pts
 			(xy 346.71 142.24) (xy 342.9 142.24)
 		)
@@
 	(wire
 		(pts
+			(xy 138.43 163.83) (xy 259.08 163.83)
+		)
+		(stroke
+			(width 0)
+			(type default)
+		)
+	)
+	(wire
+		(pts
 			(xy 381 207.01) (xy 378.46 207.01)
 		)
@@
 			)
 		)
-		(property "Value" "1n"
+		(property "Value" "330n"
 			(at 151.13 100.838 90)
 			(show_name no)

Commit message: Avances en el esquemático de Kicad.
Parts:
- removed C13: 10n, symbol Device:C
- removed R18: 1k, symbol Device:R
- removed U35: MCP4822, symbol Analog_DAC:MCP4822
Connections:
- net V_CTRL: now reaches R37.1
- net I_CTRL: now reaches R33.1
Other:
- moved on the sheet: C1, C2, C3, C37, D10, D5, D9, J1, J2, K7, Q10, Q11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
