File: Kicad/split_power_supply.kicad_sch (KiCad schematic)
At the start: 13 parts, among them Q1 NPN, Q2 PNP, Q3 NPN, Q4 PNP, Q5 NPN, U1 LM358

Commit message: Más avances en el esquemático.
Parts:
- Q1, Q5: value NPN -> 2N2222
- Q2: value PNP -> TIP36C
- Q3: value NPN -> TIP35C
- Q4: value PNP -> 2N2907
Changed lines of the file:
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@@
 		(dnp no)
 		(property "Reference" "Q2"
-			(at 210.82 72.3901 0)
-			(show_name no)
-			(do_not_autoplace no)
-			(effects
-				(font
-					(size 1.27 1.27)
-				)
-				(justify left)
-			)
-		)
-		(property "Value" "PNP"
-			(at 210.82 69.8501 0)
+			(at 210.312 67.0559 0)
+			(show_name no)
+			(do_not_autoplace no)
+			(effects
+				(font
+					(size 1.27 1.27)
+				)
+				(justify left)
+			)
+		)
+		(property "Value" "TIP36C"
+			(at 210.058 69.342 0)
 			(show_name no)
 			(do_not_autoplace no)
@@
 			)
 		)
-		(property "Value" "NPN"
+		(property "Value" "2N2222"
 			(at 199.39 80.0099 0)
 			(show_name no)
@@
 			)
 		)
-		(property "Value" "NPN"
+		(property "Value" "2N2222"
 			(at 190.5 101.5999 0)
 			(show_name no)
@@
 			)
 		)
-		(property "Value" "NPN"
+		(property "Value" "TIP35C"
 			(at 210.82 130.8099 0)
 			(show_name no)
@@
 		(dnp no)
 		(property "Reference" "Q4"
-			(at 199.39 121.9201 0)
-			(show_name no)
-			(do_not_autoplace no)
-			(effects
-				(font
-					(size 1.27 1.27)
-				)
-				(justify left)
-			)
-		)
-		(property "Value" "PNP"
+			(at 199.39 117.094 0)
+			(show_name no)
+			(do_not_autoplace no)
+			(effects
+				(font
+					(size 1.27 1.27)
+				)
+				(justify left)
+			)
+		)
+		(property "Value" "2N2907"
 			(at 199.39 119.3801 0)
 			(show_name no)
