File: Kicad/split_power_supply.kicad_sch (KiCad schematic)
At the start: 13 parts, among them Q1 NPN, Q2 PNP, Q3 NPN, Q4 PNP, Q5 NPN, U1 LM358

Commit message: Pruebas y arreglos relacionados a compensación de lazo de tensión y mediciones de frontend de módulo de carga.
Parts:
- Q1, Q5: value NPN -> 2N2222
- Q2: value PNP -> TIP36C
- Q3: value NPN -> TIP35C
- Q4: value PNP -> 2N2907
Other:
- moved on the sheet: D1, Q1, Q2, Q3, Q4, Q5, R1, R2, R3, R4, R6, RV1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
